File: esp32c3/esp32c3.kicad_pcb (KiCad board)
At the start: 0 parts

Commit message: finish first version of PCB
Parts:
- added C1: 10uF, Resistor_SMD:R_0603_1608Metric_Pad0.98x0.95mm_HandSolder, B.Cu at (37.1, 80.6)
- added C2: 0.1uF, Resistor_SMD:R_0603_1608Metric_Pad0.98x0.95mm_HandSolder, B.Cu at (39.1, 80.6)
- added C3: 10uF, Resistor_SMD:R_0603_1608Metric_Pad0.98x0.95mm_HandSolder, B.Cu at (48.3, 95.2)
- added C4: 100nF, Resistor_SMD:R_0603_1608Metric_Pad0.98x0.95mm_HandSolder, B.Cu at (41.2, 84.9)
- added C5: 100nF, Resistor_SMD:R_0603_1608Metric_Pad0.98x0.95mm_HandSolder, F.Cu at (40.1, 97.9)
- added C6: 1uF, Resistor_SMD:R_0603_1608Metric_Pad0.98x0.95mm_HandSolder, B.Cu at (42.1, 99.1)
- added C7: 1uF, Resistor_SMD:R_0603_1608Metric_Pad0.98x0.95mm_HandSolder, B.Cu at (48.9, 99.2)
- added D1: LED_RED, LED_SMD:LED_0805_2012Metric, F.Cu at (46.8, 94.2)
- added J1: A1501WR-S-2P, Connector_JST:JST_ZE_BM02B-ZESS-TBT_1x02-1MP_P1.50mm_Vertical, F.Cu at (44.9, 105.5)
- added J2: Conn_01x06, Connector_PinSocket_2.54mm:PinSocket_1x06_P2.54mm_Vertical, F.Cu at (51.8, 108.1)
- added J3: Conn_01x05, Connector_PinSocket_2.54mm:PinSocket_1x05_P2.54mm_Vertical, F.Cu at (35.1, 108.2)
- added R1: 12k, Resistor_SMD:R_0603_1608Metric_Pad0.98x0.95mm_HandSolder, B.Cu at (46.4, 95.2)
- added R10: 100k, Resistor_SMD:R_0603_1608Metric_Pad0.98x0.95mm_HandSolder, B.Cu at (34.1, 94.5)
- added R11: 100k, Resistor_SMD:R_0603_1608Metric_Pad0.98x0.95mm_HandSolder, B.Cu at (37.0, 94.6)
- added R12: 100k, Resistor_SMD:R_0603_1608Metric_Pad0.98x0.95mm_HandSolder, F.Cu at (38.0, 104.9)
- added R13: 100k, Resistor_SMD:R_0603_1608Metric_Pad0.98x0.95mm_HandSolder, F.Cu at (38.0, 108.3)
- added R2: 10k, Resistor_SMD:R_0603_1608Metric_Pad0.98x0.95mm_HandSolder, F.Cu at (44.6, 94.2)
- added R3: 10k, Resistor_SMD:R_0603_1608Metric_Pad0.98x0.95mm_HandSolder, B.Cu at (49.0, 83.3)
- added R4: 10k, Resistor_SMD:R_0603_1608Metric_Pad0.98x0.95mm_HandSolder, B.Cu at (49.0, 86.9)
- added R5: 100k, Resistor_SMD:R_0603_1608Metric_Pad0.98x0.95mm_HandSolder, B.Cu at (43.9, 95.4)
- added R6: 200k, Resistor_SMD:R_0603_1608Metric_Pad0.98x0.95mm_HandSolder, B.Cu at (42.1, 95.4)
- added R7: 5.1k, Resistor_SMD:R_0603_1608Metric_Pad0.98x0.95mm_HandSolder, B.Cu at (51.8, 92.7)
- added R8: 100k, Resistor_SMD:R_0603_1608Metric_Pad0.98x0.95mm_HandSolder, F.Cu at (37.9, 101.4)
- added R9: 100k, Resistor_SMD:R_0603_1608Metric_Pad0.98x0.95mm_HandSolder, F.Cu at (37.9, 97.9)
- added SW1: wake up, Library:SW-SMD_2PIN-L4.05-W3.00-L, F.Cu at (45.3, 98.7)
- added U1: ESP32-C3-WROOM-02, Library:ESP32-C3-WROOM-02, F.Cu at (44.3, 83.5)
- added U2: AHT10, Library:AHT10, B.Cu at (45.0, 84.4)
- added U3: LIS2DH, Package_LGA:LGA-14_2x2mm_P0.35mm_LayoutBorder3x4y, F.Cu at (40.5, 94.0)
- added U4: HX6306, Package_TO_SOT_SMD:SOT-23, B.Cu at (45.1, 99.0)
Routing:
- net 3.3V: track 0.00 -> 116.4 mm, vias 0 -> 2
- net IO2: track 0.00 -> 35.3 mm
- net EN: track 0.00 -> 31.0 mm, vias 0 -> 1
- net RXD: track 0.00 -> 28.8 mm
- net TXD: track 0.00 -> 23.5 mm
- net ADC: track 0.00 -> 23.4 mm, vias 0 -> 1
- net IO0: track 0.00 -> 23.2 mm, vias 0 -> 1
- net IO9: track 0.00 -> 22.8 mm
- net GND: track 0.00 -> 17.7 mm, vias 0 -> 12
- net LED: track 0.00 -> 17.7 mm
- net INT2: track 0.00 -> 15.1 mm
- net IO8: track 0.00 -> 15.0 mm, vias 0 -> 1
- net INT1: track 0.00 -> 13.1 mm
- net INT: track 0.00 -> 12.7 mm
- net SDA: track 0.00 -> 12.6 mm
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- added copper zone on B.Cu, net GND
- added copper zone on F.Cu, net GND
Other:
- board outline added: 20.9 x 32.9 mm
- copper layers 0 -> 2
